Commit message: Milestone1

File: body.urdf (robot description, URDF)
Before this commit: robot robot, 9 links, 8 joints
Links:
- removed link BackLeg
- removed link BackLowerLeg
- removed link FrontLeg
- removed link FrontLowerLeg
- removed link LeftLeg
- removed link LeftLowerLeg
- removed link RightLeg
- removed link RightLowerLeg
- removed link Torso
- added link BackLeg1, mass 1; collision box size=0.2 1 0.2; visual box size=0.2 1 0.2
- added link BackLeg2, mass 1; collision box size=0.2 1 0.2; visual box size=0.2 1 0.2
- added link BackLowerLeg1, mass 1; collision box size=0.2 0.2 1; visual box size=0.2 0.2 1
- added link BackLowerLeg2, mass 1; collision box size=0.2 0.2 1; visual box size=0.2 0.2 1
- added link FrontLeg1, mass 1; collision box size=0.2 1 0.2; visual box size=0.2 1 0.2
- added link FrontLeg2, mass 1; collision box size=0.2 1 0.2; visual box size=0.2 1 0.2
- added link FrontLowerLeg1, mass 1; collision box size=0.2 0.2 1; visual box size=0.2 0.2 1
- added link FrontLowerLeg2, mass 1; collision box size=0.2 0.2 1; visual box size=0.2 0.2 1
- added link Torso1, mass 1; collision box size=1 1 1; visual box size=1 1 1
- added link Torso2, mass 1; collision box size=1 1 1; visual box size=1 1 1
Joints:
- removed joint BackLeg_BackLowerLeg
- removed joint FrontLeg_FrontLowerLeg
- removed joint LeftLeg_LeftLowerLeg
- removed joint RightLeg_RightLowerLeg
- removed joint Torso_BackLeg
- removed joint Torso_FrontLeg
- removed joint Torso_LeftLeg
- removed joint Torso_RightLeg
- added joint BackLeg1_BackLowerLeg1: type revolute, parent BackLeg1, child BackLowerLeg1, origin xyz=0 -1 0 rpy=0 0 0, axis 1 0 0, limit lower=-3.14159 upper=3.14159 effort=0.0 velocity=0.0
- added joint BackLeg2_BackLowerLeg2: type revolute, parent BackLeg2, child BackLowerLeg2, origin xyz=0 -1 0 rpy=0 0 0, axis 1 0 0, limit lower=-3.14159 upper=3.14159 effort=0.0 velocity=0.0
- added joint FrontLeg1_FrontLowerLeg1: type revolute, parent FrontLeg1, child FrontLowerLeg1, origin xyz=0 1 0 rpy=0 0 0, axis 1 0 0, limit lower=-3.14159 upper=3.14159 effort=0.0 velocity=0.0
- added joint FrontLeg2_FrontLowerLeg2: type revolute, parent FrontLeg2, child FrontLowerLeg2, origin xyz=0 1 0 rpy=0 0 0, axis 1 0 0, limit lower=-3.14159 upper=3.14159 effort=0.0 velocity=0.0
- added joint Torso1_BackLeg1: type revolute, parent Torso1, child BackLeg1, origin xyz=0 -0.5 1 rpy=0 0 0, axis 1 0 0, limit lower=-3.14159 upper=3.14159 effort=0.0 velocity=0.0
- added joint Torso1_FrontLeg1: type revolute, parent Torso1, child FrontLeg1, origin xyz=0 0.5 1 rpy=0 0 0, axis 1 0 0, limit lower=-3.14159 upper=3.14159 effort=0.0 velocity=0.0
- added joint Torso1_Torso2: type revolute, parent Torso1, child Torso2, origin xyz=0 0 0 rpy=0 0 0, axis 0 1 0, limit lower=-3.14159 upper=3.14159 effort=0.0 velocity=0.0
- added joint Torso2_BackLeg2: type revolute, parent Torso2, child BackLeg2, origin xyz=0.5 -0.5 1 rpy=0 0 0, axis 1 0 0, limit lower=-3.14159 upper=3.14159 effort=0.0 velocity=0.0
- added joint Torso2_FrontLeg2: type revolute, parent Torso2, child FrontLeg2, origin xyz=0.5 0.5 1 rpy=0 0 0, axis 1 0 0, limit lower=-3.14159 upper=3.14159 effort=0.0 velocity=0.0

Commit message: Milestone2 - Changed torso, given only 2 legs so far

File: body.urdf (robot description, URDF)
Before this commit: robot robot, 10 links, 9 joints
Links:
- removed link BackLeg2
- removed link BackLowerLeg2
- removed link FrontLeg2
- removed link FrontLowerLeg2
- removed link Torso2
- link Torso1: geometry collision box size=2 1 0.5; visual box size=2 1 0.5
Joints:
- removed joint BackLeg2_BackLowerLeg2
- removed joint FrontLeg2_FrontLowerLeg2
- removed joint Torso1_Torso2
- removed joint Torso2_BackLeg2
- removed joint Torso2_FrontLeg2

Commit message: Milestone2 - 3 legs, trying to get to work. Just going to create the branches right now

File: body.urdf (robot description, URDF)
Before this commit: robot robot, 5 links, 4 joints
Links:
- added link BackLeg2, mass 1; collision box size=0.2 1 0.2; visual box size=0.2 1 0.2
- added link BackLeg3, mass 1; collision box size=0.2 1 0.2; visual box size=0.2 1 0.2
- added link BackLowerLeg2, mass 1; collision box size=0.2 0.2 1; visual box size=0.2 0.2 1
- added link BackLowerLeg3, mass 1; collision box size=0.2 0.2 1; visual box size=0.2 0.2 1
- added link FrontLeg2, mass 1; collision box size=0.2 1 0.2; visual box size=0.2 1 0.2
- added link FrontLeg3, mass 1; collision box size=0.2 1 0.2; visual box size=0.2 1 0.2
- added link FrontLowerLeg2, mass 1; collision box size=0.2 0.2 1; visual box size=0.2 0.2 1
- added link FrontLowerLeg3, mass 1; collision box size=0.2 0.2 1; visual box size=0.2 0.2 1
- link Torso1: geometry collision box size=3 1 0.5; visual box size=3 1 0.5
Joints:
- added joint BackLeg2_BackLowerLeg2: type revolute, parent BackLeg2, child BackLowerLeg2, origin xyz=0 -1 0 rpy=0 0 0, axis 1 0 0, limit lower=-3.14159 upper=3.14159 effort=0.0 velocity=0.0
- added joint BackLeg3_BackLowerLeg3: type revolute, parent BackLeg3, child BackLowerLeg3, origin xyz=0 -1 0 rpy=0 0 0, axis 1 0 0, limit lower=-3.14159 upper=3.14159 effort=0.0 velocity=0.0
- added joint FrontLeg2_FrontLowerLeg2: type revolute, parent FrontLeg2, child FrontLowerLeg2, origin xyz=0 1 0 rpy=0 0 0, axis 1 0 0, limit lower=-3.14159 upper=3.14159 effort=0.0 velocity=0.0
- added joint FrontLeg3_FrontLowerLeg3: type revolute, parent FrontLeg3, child FrontLowerLeg3, origin xyz=0 1 0 rpy=0 0 0, axis 1 0 0, limit lower=-3.14159 upper=3.14159 effort=0.0 velocity=0.0
- added joint Torso1_BackLeg2: type revolute, parent Torso1, child BackLeg2, origin xyz=0 -0.5 1 rpy=0 0 0, axis 1 1 0, limit lower=-3.14159 upper=3.14159 effort=0.0 velocity=0.0
- added joint Torso1_BackLeg3: type revolute, parent Torso1, child BackLeg3, origin xyz=0.9 -0.5 1 rpy=0 0 0, axis 1 1 0, limit lower=-3.14159 upper=3.14159 effort=0.0 velocity=0.0
- added joint Torso1_FrontLeg2: type revolute, parent Torso1, child FrontLeg2, origin xyz=0 0.5 1 rpy=0 0 0, axis 1 1 0, limit lower=-3.14159 upper=3.14159 effort=0.0 velocity=0.0
- added joint Torso1_FrontLeg3: type revolute, parent Torso1, child FrontLeg3, origin xyz=0.9 0.5 1 rpy=0 0 0, axis 1 1 0, limit lower=-3.14159 upper=3.14159 effort=0.0 velocity=0.0
- joint Torso1_BackLeg1: axis 1 0 0 -> 1 1 0; origin xyz=0 -0.5 1 rpy=0 0 0 -> xyz=-0.9 -0.5 1 rpy=0 0 0
- joint Torso1_FrontLeg1: axis 1 0 0 -> 1 1 0; origin xyz=0 0.5 1 rpy=0 0 0 -> xyz=-0.9 0.5 1 rpy=0 0 0

Commit message: Okay Awesome, 10 legs wow

File: body.urdf (robot description, URDF)
Before this commit: robot robot, 13 links, 12 joints
Links:
- added link BackLeg4, mass 1; collision box size=0.2 1 0.2; visual box size=0.2 1 0.2
- added link BackLeg5, mass 1; collision box size=0.2 1 0.2; visual box size=0.2 1 0.2
- added link BackLowerLeg4, mass 1; collision box size=0.2 0.2 1; visual box size=0.2 0.2 1
- added link BackLowerLeg5, mass 1; collision box size=0.2 0.2 1; visual box size=0.2 0.2 1
- added link FrontLeg4, mass 1; collision box size=0.2 1 0.2; visual box size=0.2 1 0.2
- added link FrontLeg5, mass 1; collision box size=0.2 1 0.2; visual box size=0.2 1 0.2
- added link FrontLowerLeg4, mass 1; collision box size=0.2 0.2 1; visual box size=0.2 0.2 1
- added link FrontLowerLeg5, mass 1; collision box size=0.2 0.2 1; visual box size=0.2 0.2 1
- link Torso1: geometry collision box size=4 1 0.5; visual box size=4 1 0.5
Joints:
- added joint BackLeg4_BackLowerLeg4: type revolute, parent BackLeg4, child BackLowerLeg4, origin xyz=0 -1 0 rpy=0 0 0, axis 1 0 0, limit lower=-3.14159 upper=3.14159 effort=0.0 velocity=0.0
- added joint BackLeg5_BackLowerLeg5: type revolute, parent BackLeg5, child BackLowerLeg5, origin xyz=0 -1 0 rpy=0 0 0, axis 1 0 0, limit lower=-3.14159 upper=3.14159 effort=0.0 velocity=0.0
- added joint FrontLeg4_FrontLowerLeg4: type revolute, parent FrontLeg4, child FrontLowerLeg4, origin xyz=0 1 0 rpy=0 0 0, axis 1 0 0, limit lower=-3.14159 upper=3.14159 effort=0.0 velocity=0.0
- added joint FrontLeg5_FrontLowerLeg5: type revolute, parent FrontLeg5, child FrontLowerLeg5, origin xyz=0 1 0 rpy=0 0 0, axis 1 0 0, limit lower=-3.14159 upper=3.14159 effort=0.0 velocity=0.0
- added joint Torso1_BackLeg4: type revolute, parent Torso1, child BackLeg4, origin xyz=0.8 -0.5 1 rpy=0 0 0, axis 1 1 0, limit lower=-3.14159 upper=3.14159 effort=0.0 velocity=0.0
- added joint Torso1_BackLeg5: type revolute, parent Torso1, child BackLeg5, origin xyz=1.6 -0.5 1 rpy=0 0 0, axis 1 1 0, limit lower=-3.14159 upper=3.14159 effort=0.0 velocity=0.0
- added joint Torso1_FrontLeg4: type revolute, parent Torso1, child FrontLeg4, origin xyz=0.8 0.5 1 rpy=0 0 0, axis 1 1 0, limit lower=-3.14159 upper=3.14159 effort=0.0 velocity=0.0
- added joint Torso1_FrontLeg5: type revolute, parent Torso1, child FrontLeg5, origin xyz=1.6 0.5 1 rpy=0 0 0, axis 1 1 0, limit lower=-3.14159 upper=3.14159 effort=0.0 velocity=0.0
- joint Torso1_BackLeg1: origin xyz=-0.9 -0.5 1 rpy=0 0 0 -> xyz=-1.6 -0.5 1 rpy=0 0 0
- joint Torso1_BackLeg2: origin xyz=0 -0.5 1 rpy=0 0 0 -> xyz=-0.8 -0.5 1 rpy=0 0 0
- joint Torso1_BackLeg3: origin xyz=0.9 -0.5 1 rpy=0 0 0 -> xyz=0.0 -0.5 1 rpy=0 0 0
- joint Torso1_FrontLeg1: origin xyz=-0.9 0.5 1 rpy=0 0 0 -> xyz=-1.6 0.5 1 rpy=0 0 0
- joint Torso1_FrontLeg2: origin xyz=0 0.5 1 rpy=0 0 0 -> xyz=-0.8 0.5 1 rpy=0 0 0
- joint Torso1_FrontLeg3: origin xyz=0.9 0.5 1 rpy=0 0 0 -> xyz=0.0 0.5 1 rpy=0 0 0

Commit message: Okay Awesome, 8 legs wow

File: body.urdf (robot description, URDF)
Before this commit: robot robot, 13 links, 12 joints
Links:
- added link BackLeg4, mass 1; collision box size=0.2 1 0.2; visual box size=0.2 1 0.2
- added link BackLowerLeg4, mass 1; collision box size=0.2 0.2 1; visual box size=0.2 0.2 1
- added link FrontLeg4, mass 1; collision box size=0.2 1 0.2; visual box size=0.2 1 0.2
- added link FrontLowerLeg4, mass 1; collision box size=0.2 0.2 1; visual box size=0.2 0.2 1
- link Torso1: geometry collision box size=3.5 1 0.5; visual box size=3.5 1 0.5
Joints:
- added joint BackLeg4_BackLowerLeg4: type revolute, parent BackLeg4, child BackLowerLeg4, origin xyz=0 -1 0 rpy=0 0 0, axis 1 0 0, limit lower=-3.14159 upper=3.14159 effort=0.0 velocity=0.0
- added joint FrontLeg4_FrontLowerLeg4: type revolute, parent FrontLeg4, child FrontLowerLeg4, origin xyz=0 1 0 rpy=0 0 0, axis 1 0 0, limit lower=-3.14159 upper=3.14159 effort=0.0 velocity=0.0
- added joint Torso1_BackLeg4: type revolute, parent Torso1, child BackLeg4, origin xyz=1.4 -0.5 1 rpy=0 0 0, axis 1 1 0, limit lower=-3.14159 upper=3.14159 effort=0.0 velocity=0.0
- added joint Torso1_FrontLeg4: type revolute, parent Torso1, child FrontLeg4, origin xyz=1.4 0.5 1 rpy=0 0 0, axis 1 1 0, limit lower=-3.14159 upper=3.14159 effort=0.0 velocity=0.0
- joint Torso1_BackLeg1: origin xyz=-0.9 -0.5 1 rpy=0 0 0 -> xyz=-1.4 -0.5 1 rpy=0 0 0
- joint Torso1_BackLeg2: origin xyz=0 -0.5 1 rpy=0 0 0 -> xyz=-0.5 -0.5 1 rpy=0 0 0
- joint Torso1_BackLeg3: origin xyz=0.9 -0.5 1 rpy=0 0 0 -> xyz=0.5 -0.5 1 rpy=0 0 0
- joint Torso1_FrontLeg1: origin xyz=-0.9 0.5 1 rpy=0 0 0 -> xyz=-1.4 0.5 1 rpy=0 0 0
- joint Torso1_FrontLeg2: origin xyz=0 0.5 1 rpy=0 0 0 -> xyz=-0.5 0.5 1 rpy=0 0 0
- joint Torso1_FrontLeg3: origin xyz=0.9 0.5 1 rpy=0 0 0 -> xyz=0.5 0.5 1 rpy=0 0 0

Commit message: Edited as I try new things

File: body.urdf (robot description, URDF)
Before this commit: robot robot, 13 links, 12 joints
Links:
- removed link BackLeg2
- removed link BackLeg3
- removed link BackLowerLeg2
- removed link BackLowerLeg3
- removed link FrontLeg2
- removed link FrontLeg3
- removed link FrontLowerLeg2
- removed link FrontLowerLeg3
Joints:
- removed joint BackLeg2_BackLowerLeg2
- removed joint BackLeg3_BackLowerLeg3
- removed joint FrontLeg2_FrontLowerLeg2
- removed joint FrontLeg3_FrontLowerLeg3
- removed joint Torso1_BackLeg2
- removed joint Torso1_BackLeg3
- removed joint Torso1_FrontLeg2
- removed joint Torso1_FrontLeg3

Commit message: Trying to get front legs to work properly

File: body.urdf (robot description, URDF)
Before this commit: robot robot, 9 links, 8 joints
Links:
- removed link BackLeg
- removed link BackLowerLeg
- removed link FrontLeg
- removed link FrontLowerLeg
- removed link LeftLeg
- removed link LeftLowerLeg
- removed link RightLeg
- removed link RightLowerLeg
- removed link Torso
- added link BackLeg1, mass 1; collision box size=0.2 1 0.2; visual box size=0.2 1 0.2
- added link BackLeg2, mass 1; collision box size=0.2 1 0.2; visual box size=0.2 1 0.2
- added link BackLowerLeg1, mass 1; collision box size=0.2 0.2 1; visual box size=0.2 0.2 1
- added link BackLowerLeg2, mass 1; collision box size=0.2 0.2 1; visual box size=0.2 0.2 1
- added link FrontLeg1, mass 1; collision box size=0.2 1 0.2; visual box size=0.2 1 0.2
- added link FrontLeg2, mass 1; collision box size=0.2 1 0.2; visual box size=0.2 1 0.2
- added link FrontLowerLeg1, mass 1; collision box size=0.2 0.2 1; visual box size=0.2 0.2 1
- added link FrontLowerLeg2, mass 1; collision box size=0.2 0.2 1; visual box size=0.2 0.2 1
- added link Torso1, mass 1; collision box size=2 1 0.5; visual box size=2 1 0.5
Joints:
- removed joint BackLeg_BackLowerLeg
- removed joint FrontLeg_FrontLowerLeg
- removed joint LeftLeg_LeftLowerLeg
- removed joint RightLeg_RightLowerLeg
- removed joint Torso_BackLeg
- removed joint Torso_FrontLeg
- removed joint Torso_LeftLeg
- removed joint Torso_RightLeg
- added joint BackLeg1_BackLowerLeg1: type revolute, parent BackLeg1, child BackLowerLeg1, origin xyz=0 -1 0 rpy=0 0 0, axis 1 0 0, limit lower=-3.14159 upper=3.14159 effort=0.0 velocity=0.0
- added joint BackLeg2_BackLowerLeg2: type revolute, parent BackLeg2, child BackLowerLeg2, origin xyz=0 -1 0 rpy=0 0 0, axis 1 0 0, limit lower=-3.14159 upper=3.14159 effort=0.0 velocity=0.0
- added joint FrontLeg1_FrontLowerLeg1: type revolute, parent FrontLeg1, child FrontLowerLeg1, origin xyz=0 1 0 rpy=0 0 0, axis 1 0 0, limit lower=-3.14159 upper=3.14159 effort=0.0 velocity=0.0
- added joint FrontLeg2_FrontLowerLeg2: type revolute, parent FrontLeg2, child FrontLowerLeg2, origin xyz=0 1 0 rpy=0 0 0, axis 1 0 0, limit lower=-3.14159 upper=3.14159 effort=0.0 velocity=0.0
- added joint Torso1_BackLeg1: type revolute, parent Torso1, child BackLeg1, origin xyz=-0.9 -0.5 1 rpy=0 0 0, axis 1 1 0, limit lower=-3.14159 upper=3.14159 effort=0.0 velocity=0.0
- added joint Torso1_BackLeg2: type revolute, parent Torso1, child BackLeg2, origin xyz=0 -0.5 1 rpy=0 0 0, axis 1 1 0, limit lower=-3.14159 upper=3.14159 effort=0.0 velocity=0.0
- added joint Torso1_FrontLeg1: type revolute, parent Torso1, child FrontLeg1, origin xyz=-0.9 0.5 1 rpy=0 0 0, axis 1 1 0, limit lower=-3.14159 upper=3.14159 effort=0.0 velocity=0.0
- added joint Torso1_FrontLeg2: type revolute, parent Torso1, child FrontLeg2, origin xyz=0 0.5 1 rpy=0 0 0, axis 1 1 0, limit lower=-3.14159 upper=3.14159 effort=0.0 velocity=0.0

Commit message: Synchro for 3 legs

File: body.urdf (robot description, URDF)
Before this commit: robot robot, 9 links, 8 joints
Links:
- removed link BackLeg1
- removed link BackLeg2
- removed link BackLowerLeg1
- removed link BackLowerLeg2
- removed link FrontLeg1
- removed link FrontLeg2
- removed link FrontLowerLeg1
- removed link FrontLowerLeg2
- added link LeftLeg1, mass 1; collision box size=0.2 1 0.2; visual box size=0.2 1 0.2
- added link LeftLeg2, mass 1; collision box size=0.2 1 0.2; visual box size=0.2 1 0.2
- added link LeftLeg3, mass 1; collision box size=0.2 1 0.2; visual box size=0.2 1 0.2
- added link LeftLowerLeg1, mass 1; collision box size=0.2 0.2 1; visual box size=0.2 0.2 1
- added link LeftLowerLeg2, mass 1; collision box size=0.2 0.2 1; visual box size=0.2 0.2 1
- added link LeftLowerLeg3, mass 1; collision box size=0.2 0.2 1; visual box size=0.2 0.2 1
- added link RightLeg1, mass 1; collision box size=0.2 1 0.2; visual box size=0.2 1 0.2
- added link RightLeg2, mass 1; collision box size=0.2 1 0.2; visual box size=0.2 1 0.2
- added link RightLeg3, mass 1; collision box size=0.2 1 0.2; visual box size=0.2 1 0.2
- added link RightLowerLeg1, mass 1; collision box size=0.2 0.2 1; visual box size=0.2 0.2 1
- added link RightLowerLeg2, mass 1; collision box size=0.2 0.2 1; visual box size=0.2 0.2 1
- added link RightLowerLeg3, mass 1; collision box size=0.2 0.2 1; visual box size=0.2 0.2 1
- link Torso1: geometry collision box size=3 1 0.5; visual box size=3 1 0.5
Joints:
- removed joint BackLeg1_BackLowerLeg1
- removed joint BackLeg2_BackLowerLeg2
- removed joint FrontLeg1_FrontLowerLeg1
- removed joint FrontLeg2_FrontLowerLeg2
- removed joint Torso1_BackLeg1
- removed joint Torso1_BackLeg2
- removed joint Torso1_FrontLeg1
- removed joint Torso1_FrontLeg2
- added joint LeftLeg1_LeftLowerLeg1: type revolute, parent LeftLeg1, child LeftLowerLeg1, origin xyz=0 -1 0 rpy=0 0 0, axis 1 0 0, limit lower=-3.14159 upper=3.14159 effort=0.0 velocity=0.0
- added joint LeftLeg2_LeftLowerLeg2: type revolute, parent LeftLeg2, child LeftLowerLeg2, origin xyz=0 -1 0 rpy=0 0 0, axis 1 0 0, limit lower=-3.14159 upper=3.14159 effort=0.0 velocity=0.0
- added joint LeftLeg3_LeftLowerLeg3: type revolute, parent LeftLeg3, child LeftLowerLeg3, origin xyz=0 -1 0 rpy=0 0 0, axis 1 0 0, limit lower=-3.14159 upper=3.14159 effort=0.0 velocity=0.0
- added joint RightLeg1_RightLowerLeg1: type revolute, parent RightLeg1, child RightLowerLeg1, origin xyz=0 1 0 rpy=0 0 0, axis 1 0 0, limit lower=-3.14159 upper=3.14159 effort=0.0 velocity=0.0
- added joint RightLeg2_RightLowerLeg2: type revolute, parent RightLeg2, child RightLowerLeg2, origin xyz=0 1 0 rpy=0 0 0, axis 1 0 0, limit lower=-3.14159 upper=3.14159 effort=0.0 velocity=0.0
- added joint RightLeg3_RightLowerLeg3: type revolute, parent RightLeg3, child RightLowerLeg3, origin xyz=0 1 0 rpy=0 0 0, axis 1 0 0, limit lower=-3.14159 upper=3.14159 effort=0.0 velocity=0.0
- added joint Torso1_LeftLeg1: type revolute, parent Torso1, child LeftLeg1, origin xyz=-0.9 -0.5 1 rpy=0 0 0, axis 1 1 0, limit lower=-3.14159 upper=3.14159 effort=0.0 velocity=0.0
- added joint Torso1_LeftLeg2: type revolute, parent Torso1, child LeftLeg2, origin xyz=0 -0.5 1 rpy=0 0 0, axis 1 1 0, limit lower=-3.14159 upper=3.14159 effort=0.0 velocity=0.0
- added joint Torso1_LeftLeg3: type revolute, parent Torso1, child LeftLeg3, origin xyz=0.9 -0.5 1 rpy=0 0 0, axis 1 1 0, limit lower=-3.14159 upper=3.14159 effort=0.0 velocity=0.0
- added joint Torso1_RightLeg1: type revolute, parent Torso1, child RightLeg1, origin xyz=-0.9 0.5 1 rpy=0 0 0, axis 1 1 0, limit lower=-3.14159 upper=3.14159 effort=0.0 velocity=0.0
- added joint Torso1_RightLeg2: type revolute, parent Torso1, child RightLeg2, origin xyz=0 0.5 1 rpy=0 0 0, axis 1 1 0, limit lower=-3.14159 upper=3.14159 effort=0.0 velocity=0.0
- added joint Torso1_RightLeg3: type revolute, parent Torso1, child RightLeg3, origin xyz=0.9 0.5 1 rpy=0 0 0, axis 1 1 0, limit lower=-3.14159 upper=3.14159 effort=0.0 velocity=0.0
