Commit message: Synchro for 4 legs

File: body.urdf (robot description, URDF)
Before this commit: robot robot, 9 links, 8 joints
Links:
- removed link BackLeg1
- removed link BackLeg2
- removed link BackLowerLeg1
- removed link BackLowerLeg2
- removed link FrontLeg1
- removed link FrontLeg2
- removed link FrontLowerLeg1
- removed link FrontLowerLeg2
- added link LeftLeg1, mass 1; collision box size=0.2 1 0.2; visual box size=0.2 1 0.2
- added link LeftLeg2, mass 1; collision box size=0.2 1 0.2; visual box size=0.2 1 0.2
- added link LeftLeg3, mass 1; collision box size=0.2 1 0.2; visual box size=0.2 1 0.2
- added link LeftLeg4, mass 1; collision box size=0.2 1 0.2; visual box size=0.2 1 0.2
- added link LeftLowerLeg1, mass 1; collision box size=0.2 0.2 1; visual box size=0.2 0.2 1
- added link LeftLowerLeg2, mass 1; collision box size=0.2 0.2 1; visual box size=0.2 0.2 1
- added link LeftLowerLeg3, mass 1; collision box size=0.2 0.2 1; visual box size=0.2 0.2 1
- added link LeftLowerLeg4, mass 1; collision box size=0.2 0.2 1; visual box size=0.2 0.2 1
- added link RightLeg1, mass 1; collision box size=0.2 1 0.2; visual box size=0.2 1 0.2
- added link RightLeg2, mass 1; collision box size=0.2 1 0.2; visual box size=0.2 1 0.2
- added link RightLeg3, mass 1; collision box size=0.2 1 0.2; visual box size=0.2 1 0.2
- added link RightLeg4, mass 1; collision box size=0.2 1 0.2; visual box size=0.2 1 0.2
- added link RightLowerLeg1, mass 1; collision box size=0.2 0.2 1; visual box size=0.2 0.2 1
- added link RightLowerLeg2, mass 1; collision box size=0.2 0.2 1; visual box size=0.2 0.2 1
- added link RightLowerLeg3, mass 1; collision box size=0.2 0.2 1; visual box size=0.2 0.2 1
- added link RightLowerLeg4, mass 1; collision box size=0.2 0.2 1; visual box size=0.2 0.2 1
- link Torso1: geometry collision box size=3.5 1 0.5; visual box size=3.5 1 0.5
Joints:
- removed joint BackLeg1_BackLowerLeg1
- removed joint BackLeg2_BackLowerLeg2
- removed joint FrontLeg1_FrontLowerLeg1
- removed joint FrontLeg2_FrontLowerLeg2
- removed joint Torso1_BackLeg1
- removed joint Torso1_BackLeg2
- removed joint Torso1_FrontLeg1
- removed joint Torso1_FrontLeg2
- added joint LeftLeg1_LeftLowerLeg1: type revolute, parent LeftLeg1, child LeftLowerLeg1, origin xyz=0 -1 0 rpy=0 0 0, axis 1 0 0, limit lower=-3.14159 upper=3.14159 effort=0.0 velocity=0.0
- added joint LeftLeg2_LeftLowerLeg2: type revolute, parent LeftLeg2, child LeftLowerLeg2, origin xyz=0 -1 0 rpy=0 0 0, axis 1 0 0, limit lower=-3.14159 upper=3.14159 effort=0.0 velocity=0.0
- added joint LeftLeg3_LeftLowerLeg3: type revolute, parent LeftLeg3, child LeftLowerLeg3, origin xyz=0 -1 0 rpy=0 0 0, axis 1 0 0, limit lower=-3.14159 upper=3.14159 effort=0.0 velocity=0.0
- added joint LeftLeg4_LeftLowerLeg4: type revolute, parent LeftLeg4, child LeftLowerLeg4, origin xyz=0 -1 0 rpy=0 0 0, axis 1 0 0, limit lower=-3.14159 upper=3.14159 effort=0.0 velocity=0.0
- added joint RightLeg1_RightLowerLeg1: type revolute, parent RightLeg1, child RightLowerLeg1, origin xyz=0 1 0 rpy=0 0 0, axis 1 0 0, limit lower=-3.14159 upper=3.14159 effort=0.0 velocity=0.0
- added joint RightLeg2_RightLowerLeg2: type revolute, parent RightLeg2, child RightLowerLeg2, origin xyz=0 1 0 rpy=0 0 0, axis 1 0 0, limit lower=-3.14159 upper=3.14159 effort=0.0 velocity=0.0
- added joint RightLeg3_RightLowerLeg3: type revolute, parent RightLeg3, child RightLowerLeg3, origin xyz=0 1 0 rpy=0 0 0, axis 1 0 0, limit lower=-3.14159 upper=3.14159 effort=0.0 velocity=0.0
- added joint RightLeg4_RightLowerLeg4: type revolute, parent RightLeg4, child RightLowerLeg4, origin xyz=0 1 0 rpy=0 0 0, axis 1 0 0, limit lower=-3.14159 upper=3.14159 effort=0.0 velocity=0.0
- added joint Torso1_LeftLeg1: type revolute, parent Torso1, child LeftLeg1, origin xyz=-0.9 -0.5 1 rpy=0 0 0, axis 1 1 0, limit lower=-3.14159 upper=3.14159 effort=0.0 velocity=0.0
- added joint Torso1_LeftLeg2: type revolute, parent Torso1, child LeftLeg2, origin xyz=0 -0.5 1 rpy=0 0 0, axis 1 1 0, limit lower=-3.14159 upper=3.14159 effort=0.0 velocity=0.0
- added joint Torso1_LeftLeg3: type revolute, parent Torso1, child LeftLeg3, origin xyz=0.9 -0.5 1 rpy=0 0 0, axis 1 1 0, limit lower=-3.14159 upper=3.14159 effort=0.0 velocity=0.0
- added joint Torso1_LeftLeg4: type revolute, parent Torso1, child LeftLeg4, origin xyz=1.4 -0.5 1 rpy=0 0 0, axis 1 1 0, limit lower=-3.14159 upper=3.14159 effort=0.0 velocity=0.0
- added joint Torso1_RightLeg1: type revolute, parent Torso1, child RightLeg1, origin xyz=-0.9 0.5 1 rpy=0 0 0, axis 1 1 0, limit lower=-3.14159 upper=3.14159 effort=0.0 velocity=0.0
- added joint Torso1_RightLeg2: type revolute, parent Torso1, child RightLeg2, origin xyz=0 0.5 1 rpy=0 0 0, axis 1 1 0, limit lower=-3.14159 upper=3.14159 effort=0.0 velocity=0.0
- added joint Torso1_RightLeg3: type revolute, parent Torso1, child RightLeg3, origin xyz=0.9 0.5 1 rpy=0 0 0, axis 1 1 0, limit lower=-3.14159 upper=3.14159 effort=0.0 velocity=0.0
- added joint Torso1_RightLeg4: type revolute, parent Torso1, child RightLeg4, origin xyz=1.4 0.5 1 rpy=0 0 0, axis 1 1 0, limit lower=-3.14159 upper=3.14159 effort=0.0 velocity=0.0

Commit message: Changed names, changed size of legs back

File: body.urdf (robot description, URDF)
Before this commit: robot robot, 9 links, 8 joints
Links:
- removed link BackLeg1
- removed link BackLeg2
- removed link BackLowerLeg1
- removed link BackLowerLeg2
- removed link FrontLeg1
- removed link FrontLeg2
- removed link FrontLowerLeg1
- removed link FrontLowerLeg2
- added link LeftLeg1, mass 1; collision box size=0.2 1 0.2; visual box size=0.2 1 0.2
- added link LeftLeg2, mass 1; collision box size=0.2 1 0.2; visual box size=0.2 1 0.2
- added link LeftLowerLeg1, mass 1; collision box size=0.2 0.2 1; visual box size=0.2 0.2 1
- added link LeftLowerLeg2, mass 1; collision box size=0.2 0.2 1; visual box size=0.2 0.2 1
- added link RightLeg1, mass 1; collision box size=0.2 1 0.2; visual box size=0.2 1 0.2
- added link RightLeg2, mass 1; collision box size=0.2 1 0.2; visual box size=0.2 1 0.2
- added link RightLowerLeg1, mass 1; collision box size=0.2 0.2 1; visual box size=0.2 0.2 1
- added link RightLowerLeg2, mass 1; collision box size=0.2 0.2 1; visual box size=0.2 0.2 1
Joints:
- removed joint BackLeg1_BackLowerLeg1
- removed joint BackLeg2_BackLowerLeg2
- removed joint FrontLeg1_FrontLowerLeg1
- removed joint FrontLeg2_FrontLowerLeg2
- removed joint Torso1_BackLeg1
- removed joint Torso1_BackLeg2
- removed joint Torso1_FrontLeg1
- removed joint Torso1_FrontLeg2
- added joint LeftLeg1_LeftLowerLeg1: type revolute, parent LeftLeg1, child LeftLowerLeg1, origin xyz=0 -1 0 rpy=0 0 0, axis 0 1 0, limit lower=-3.14159 upper=3.14159 effort=0.0 velocity=0.0
- added joint LeftLeg2_LeftLowerLeg2: type revolute, parent LeftLeg2, child LeftLowerLeg2, origin xyz=0 -1 0 rpy=0 0 0, axis 0 1 0, limit lower=-3.14159 upper=3.14159 effort=0.0 velocity=0.0
- added joint RightLeg1_RightLowerLeg1: type revolute, parent RightLeg1, child RightLowerLeg1, origin xyz=0 1 0 rpy=0 0 0, axis 0 1 0, limit lower=-3.14159 upper=3.14159 effort=0.0 velocity=0.0
- added joint RightLeg2_RightLowerLeg2: type revolute, parent RightLeg2, child RightLowerLeg2, origin xyz=0 1 0 rpy=0 0 0, axis 0 1 0, limit lower=-3.14159 upper=3.14159 effort=0.0 velocity=0.0
- added joint Torso1_LeftLeg1: type revolute, parent Torso1, child LeftLeg1, origin xyz=-0.9 -0.5 1 rpy=0 0 0, axis 1 0 1, limit lower=-3.14159 upper=3.14159 effort=0.0 velocity=0.0
- added joint Torso1_LeftLeg2: type revolute, parent Torso1, child LeftLeg2, origin xyz=0.4 -0.5 1 rpy=0 0 0, axis 1 0 1, limit lower=-3.14159 upper=3.14159 effort=0.0 velocity=0.0
- added joint Torso1_RightLeg1: type revolute, parent Torso1, child RightLeg1, origin xyz=-0.9 0.5 1 rpy=0 0 0, axis 1 0 1, limit lower=-3.14159 upper=3.14159 effort=0.0 velocity=0.0
- added joint Torso1_RightLeg2: type revolute, parent Torso1, child RightLeg2, origin xyz=0.4 0.5 1 rpy=0 0 0, axis 1 0 1, limit lower=-3.14159 upper=3.14159 effort=0.0 velocity=0.0

Commit message: fitness function now rewards for time, propultion, and penalized tilt and energy use

File: body.urdf (robot description, URDF)
Before this commit: robot robot, 13 links, 12 joints
Joints:
- joint LeftLeg1_LeftLowerLeg1: axis 1 0 0 -> 0 1 0
- joint LeftLeg2_LeftLowerLeg2: axis 1 0 0 -> 0 1 0
- joint LeftLeg3_LeftLowerLeg3: axis 1 0 0 -> 0 1 0
- joint RightLeg1_RightLowerLeg1: axis 1 0 0 -> 0 1 0
- joint RightLeg2_RightLowerLeg2: axis 1 0 0 -> 0 1 0
- joint RightLeg3_RightLowerLeg3: axis 1 0 0 -> 0 1 0
- joint Torso1_LeftLeg1: axis 1 1 0 -> 1 0 1
- joint Torso1_LeftLeg2: axis 1 1 0 -> 1 0 1
- joint Torso1_LeftLeg3: axis 1 1 0 -> 1 0 1
- joint Torso1_RightLeg1: axis 1 1 0 -> 1 0 1
- joint Torso1_RightLeg2: axis 1 1 0 -> 1 0 1
- joint Torso1_RightLeg3: axis 1 1 0 -> 1 0 1

Commit message: Okay, this is the best its been

File: body.urdf (robot description, URDF)
Before this commit: robot robot, 13 links, 12 joints
Links:
- removed link LeftLeg3
- removed link LeftLowerLeg3
- removed link RightLeg3
- removed link RightLowerLeg3
- link Torso1: geometry collision box size=2 1 0.5; visual box size=2 1 0.5
Joints:
- removed joint LeftLeg3_LeftLowerLeg3
- removed joint RightLeg3_RightLowerLeg3
- removed joint Torso1_LeftLeg3
- removed joint Torso1_RightLeg3
- joint Torso1_LeftLeg2: origin xyz=0 -0.5 1 rpy=0 0 0 -> xyz=0.4 -0.5 1 rpy=0 0 0
- joint Torso1_RightLeg2: origin xyz=0 0.5 1 rpy=0 0 0 -> xyz=0.4 0.5 1 rpy=0 0 0

Commit message: Fixed (mostly)

File: body.urdf (robot description, URDF)
Before this commit: robot robot, 9 links, 8 joints
Links:
- added link LeftLeg3, mass 1; collision box size=0.2 1 0.2; visual box size=0.2 1 0.2
- added link LeftLeg4, mass 1; collision box size=0.2 1 0.2; visual box size=0.2 1 0.2
- added link LeftLowerLeg3, mass 1; collision box size=0.2 0.2 1; visual box size=0.2 0.2 1
- added link LeftLowerLeg4, mass 1; collision box size=0.2 0.2 1; visual box size=0.2 0.2 1
- added link RightLeg3, mass 1; collision box size=0.2 1 0.2; visual box size=0.2 1 0.2
- added link RightLeg4, mass 1; collision box size=0.2 1 0.2; visual box size=0.2 1 0.2
- added link RightLowerLeg3, mass 1; collision box size=0.2 0.2 1; visual box size=0.2 0.2 1
- added link RightLowerLeg4, mass 1; collision box size=0.2 0.2 1; visual box size=0.2 0.2 1
- link Torso1: geometry collision box size=3.5 1 0.5; visual box size=3.5 1 0.5
Joints:
- added joint LeftLeg3_LeftLowerLeg3: type revolute, parent LeftLeg3, child LeftLowerLeg3, origin xyz=0 -1 0 rpy=0 0 0, axis 1 0 0, limit lower=-3.14159 upper=3.14159 effort=0.0 velocity=0.0
- added joint LeftLeg4_LeftLowerLeg4: type revolute, parent LeftLeg4, child LeftLowerLeg4, origin xyz=0 -1 0 rpy=0 0 0, axis 1 0 0, limit lower=-3.14159 upper=3.14159 effort=0.0 velocity=0.0
- added joint RightLeg3_RightLowerLeg3: type revolute, parent RightLeg3, child RightLowerLeg3, origin xyz=0 1 0 rpy=0 0 0, axis 1 0 0, limit lower=-3.14159 upper=3.14159 effort=0.0 velocity=0.0
- added joint RightLeg4_RightLowerLeg4: type revolute, parent RightLeg4, child RightLowerLeg4, origin xyz=0 1 0 rpy=0 0 0, axis 1 0 0, limit lower=-3.14159 upper=3.14159 effort=0.0 velocity=0.0
- added joint Torso1_LeftLeg3: type revolute, parent Torso1, child LeftLeg3, origin xyz=0.9 -0.5 1 rpy=0 0 0, axis 1 1 0, limit lower=-3.14159 upper=3.14159 effort=0.0 velocity=0.0
- added joint Torso1_LeftLeg4: type revolute, parent Torso1, child LeftLeg4, origin xyz=1.4 -0.5 1 rpy=0 0 0, axis 1 1 0, limit lower=-3.14159 upper=3.14159 effort=0.0 velocity=0.0
- added joint Torso1_RightLeg3: type revolute, parent Torso1, child RightLeg3, origin xyz=0.9 0.5 1 rpy=0 0 0, axis 1 1 0, limit lower=-3.14159 upper=3.14159 effort=0.0 velocity=0.0
- added joint Torso1_RightLeg4: type revolute, parent Torso1, child RightLeg4, origin xyz=1.4 0.5 1 rpy=0 0 0, axis 1 1 0, limit lower=-3.14159 upper=3.14159 effort=0.0 velocity=0.0
- joint Torso1_LeftLeg2: origin xyz=0.4 -0.5 1 rpy=0 0 0 -> xyz=0 -0.5 1 rpy=0 0 0
- joint Torso1_RightLeg2: origin xyz=0.4 0.5 1 rpy=0 0 0 -> xyz=0 0.5 1 rpy=0 0 0

Commit message: TA Help

File: body.urdf (robot description, URDF)
Before this commit: robot robot, 13 links, 12 joints
Joints:
- joint Torso1_LeftLeg1: axis 1 0 1 -> 1 0 0
- joint Torso1_LeftLeg2: axis 1 0 1 -> 1 0 0
- joint Torso1_LeftLeg3: axis 1 0 1 -> 1 0 0
- joint Torso1_RightLeg1: axis 1 0 1 -> 1 0 0
- joint Torso1_RightLeg2: axis 1 0 1 -> 1 0 0
- joint Torso1_RightLeg3: axis 1 0 1 -> 1 0 0

Commit message: TA Help

File: body.urdf (robot description, URDF)
Before this commit: robot robot, 13 links, 12 joints
Links:
- removed link LeftLeg3
- removed link LeftLowerLeg3
- removed link RightLeg3
- removed link RightLowerLeg3
- link Torso1: geometry collision box size=2 1 0.5; visual box size=2 1 0.5
Joints:
- removed joint LeftLeg3_LeftLowerLeg3
- removed joint RightLeg3_RightLowerLeg3
- removed joint Torso1_LeftLeg3
- removed joint Torso1_RightLeg3
- joint Torso1_LeftLeg1: axis 1 0 0 -> 1 0 1
- joint Torso1_LeftLeg2: axis 1 0 0 -> 1 0 1; origin xyz=0 -0.5 1 rpy=0 0 0 -> xyz=0.4 -0.5 1 rpy=0 0 0
- joint Torso1_RightLeg1: axis 1 0 0 -> 1 0 1
- joint Torso1_RightLeg2: axis 1 0 0 -> 1 0 1; origin xyz=0 0.5 1 rpy=0 0 0 -> xyz=0.4 0.5 1 rpy=0 0 0

Commit message: TA Help
Signed-off-by: Sam <sdwill@uvm.edu>

File: body.urdf (robot description, URDF)
Before this commit: robot robot, 9 links, 8 joints
Links:
- added link LeftLeg3, mass 1; collision box size=0.2 1 0.2; visual box size=0.2 1 0.2
- added link LeftLowerLeg3, mass 1; collision box size=0.2 0.2 1; visual box size=0.2 0.2 1
- added link RightLeg3, mass 1; collision box size=0.2 1 0.2; visual box size=0.2 1 0.2
- added link RightLowerLeg3, mass 1; collision box size=0.2 0.2 1; visual box size=0.2 0.2 1
- link Torso1: geometry collision box size=3 1 0.5; visual box size=3 1 0.5
Joints:
- added joint LeftLeg3_LeftLowerLeg3: type revolute, parent LeftLeg3, child LeftLowerLeg3, origin xyz=0 -1 0 rpy=0 0 0, axis 0 1 0, limit lower=-3.14159 upper=3.14159 effort=0.0 velocity=0.0
- added joint RightLeg3_RightLowerLeg3: type revolute, parent RightLeg3, child RightLowerLeg3, origin xyz=0 1 0 rpy=0 0 0, axis 0 1 0, limit lower=-3.14159 upper=3.14159 effort=0.0 velocity=0.0
- added joint Torso1_LeftLeg3: type revolute, parent Torso1, child LeftLeg3, origin xyz=0.9 -0.5 1 rpy=0 0 0, axis 1 0 0, limit lower=-3.14159 upper=3.14159 effort=0.0 velocity=0.0
- added joint Torso1_RightLeg3: type revolute, parent Torso1, child RightLeg3, origin xyz=0.9 0.5 1 rpy=0 0 0, axis 1 0 0, limit lower=-3.14159 upper=3.14159 effort=0.0 velocity=0.0
- joint Torso1_LeftLeg1: axis 1 0 1 -> 1 0 0
- joint Torso1_LeftLeg2: axis 1 0 1 -> 1 0 0; origin xyz=0.4 -0.5 1 rpy=0 0 0 -> xyz=0 -0.5 1 rpy=0 0 0
- joint Torso1_RightLeg1: axis 1 0 1 -> 1 0 0
- joint Torso1_RightLeg2: axis 1 0 1 -> 1 0 0; origin xyz=0.4 0.5 1 rpy=0 0 0 -> xyz=0 0.5 1 rpy=0 0 0

Commit message: Fitness Function wrong?
Signed-off-by: Sam <sdwill@uvm.edu>

File: body.urdf (robot description, URDF)
Before this commit: robot robot, 17 links, 16 joints
Joints:
- joint LeftLeg3_LeftLowerLeg3: axis 1 0 0 -> 0 1 0
- joint LeftLeg4_LeftLowerLeg4: axis 1 0 0 -> 0 1 0
- joint RightLeg3_RightLowerLeg3: axis 1 0 0 -> 0 1 0
- joint RightLeg4_RightLowerLeg4: axis 1 0 0 -> 0 1 0
- joint Torso1_LeftLeg1: axis 1 0 1 -> 1 0 0
- joint Torso1_LeftLeg2: axis 1 0 1 -> 1 0 0
- joint Torso1_LeftLeg4: axis 1 1 0 -> 1 0 0
- joint Torso1_RightLeg1: axis 1 0 1 -> 1 0 0
- joint Torso1_RightLeg2: axis 1 0 1 -> 1 0 0
- joint Torso1_RightLeg3: axis 1 1 0 -> 1 0 0
- joint Torso1_RightLeg4: axis 1 1 0 -> 1 0 0

Commit message: Update fitness funciton
Signed-off-by: Sam <sdwill@uvm.edu>

File: body.urdf (robot description, URDF)
Before this commit: robot robot, 9 links, 8 joints
Joints:
- joint Torso1_LeftLeg1: origin xyz=-0.9 -0.5 1 rpy=0 0 0 -> xyz=-0.75 -0.5 1 rpy=0 0 0
- joint Torso1_LeftLeg2: origin xyz=0.4 -0.5 1 rpy=0 0 0 -> xyz=0.75 -0.5 1 rpy=0 0 0
- joint Torso1_RightLeg1: origin xyz=-0.9 0.5 1 rpy=0 0 0 -> xyz=-0.75 0.5 1 rpy=0 0 0
- joint Torso1_RightLeg2: origin xyz=0.4 0.5 1 rpy=0 0 0 -> xyz=0.75 0.5 1 rpy=0 0 0

Commit message: to show prof.
Signed-off-by: Sam <sdwill@uvm.edu>

File: body.urdf (robot description, URDF)
Before this commit: robot robot, 9 links, 8 joints
Joints:
- joint Torso1_LeftLeg1: axis 1 0 1 -> 1 0 0
- joint Torso1_LeftLeg2: axis 1 0 1 -> 1 0 0
- joint Torso1_RightLeg1: axis 1 0 1 -> 1 0 0
- joint Torso1_RightLeg2: axis 1 0 1 -> 1 0 0

Commit message: Somehtings wrong, can't remove limbs

File: body.urdf (robot description, URDF)
Before this commit: robot robot, 9 links, 8 joints
Links:
- removed link LeftLeg2
- removed link LeftLowerLeg2
Joints:
- removed joint LeftLeg2_LeftLowerLeg2
- removed joint Torso1_LeftLeg2

Commit message: This one works tho

File: body.urdf (robot description, URDF)
Before this commit: robot robot, 13 links, 12 joints
Links:
- removed link LeftLowerLeg3
Joints:
- removed joint LeftLeg3_LeftLowerLeg3

Commit message: Ok what the math

File: body.urdf (robot description, URDF)
Before this commit: robot robot, 9 links, 8 joints
Links:
- removed link LeftLowerLeg2
Joints:
- removed joint LeftLeg2_LeftLowerLeg2
